File: HDK/MecatronPDU-HV.kicad_pcb (KiCad board)
At the start: 2 copper layers, 80 x 80 mm, 41 parts, among them J101 Power In, J102 V_{Comp}, J106 E-Stops, J201 Power Out, J202 Power Out, J203 Power Out, J204 Power Out, J205 Power Out, J206 Power Out, J207 Power Out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

Commit message: init v2
Parts:
- removed F101: Fuse, lib:FUSE-MCCQ-122
- removed J106: E-Stops, lib:PinHeader_2x03_P2.54mm_Vertical
- added J103: E-Stops, lib:PinHeader_2x03_P2.54mm_Vertical, F.Cu at (94.5, 146.3)
- added J104: Voltmeter Probe, lib:JST_XH_B2B-XH-AM_1x02_P2.50mm_Vertical, F.Cu at (2.75, 23.5)
- added J202: Power Out, lib:AMASS_XT30U-M_1x02_P5.0mm_Vertical, F.Cu at (107.2, 115.2)
- added J202: Power Out, lib:AMASS_XT30U-M_1x02_P5.0mm_Vertical, F.Cu at (107.2, 100.8)
- added J210: 12v Out, lib:AMASS_XT30U-M_1x02_P5.0mm_Vertical, F.Cu at (-21.9, 36.0)
- added J211: 12v Out, lib:AMASS_XT30U-M_1x02_P5.0mm_Vertical, F.Cu at (-21.9, 43.2)
- added J212: 12v Out, Connector_PinHeader_2.54mm:PinHeader_2x04_P2.54mm_Vertical, F.Cu at (-23.2, 22.4)
- added J213: 5v Out, Connector_PinHeader_2.54mm:PinHeader_2x04_P2.54mm_Vertical, F.Cu at (-16.1, 22.4)
- added REF**: AMASS_XT30PW-M_1x02_P2.50mm_Horizontal, Connector_AMASS:AMASS_XT30PW-M_1x02_P2.50mm_Horizontal, F.Cu at (64.2, 65.5)
- added REF**: AMASS_XT30PW-M_1x02_P2.50mm_Horizontal, Connector_AMASS:AMASS_XT30PW-M_1x02_P2.50mm_Horizontal, F.Cu at (64.2, 80.0)
- added REF**: AMASS_XT30PW-M_1x02_P2.50mm_Horizontal, Connector_AMASS:AMASS_XT30PW-M_1x02_P2.50mm_Horizontal, F.Cu at (116.0, 115.5)
- added REF**: FUSE-MCCQ-121, lib:FUSE-MCCQ-121, F.Cu at (89.0, 139.8)
- added REF**: AMASS_XT30PW-M_1x02_P2.50mm_Horizontal, Connector_AMASS:AMASS_XT30PW-M_1x02_P2.50mm_Horizontal, F.Cu at (116.0, 72.0)
- added REF**: AMASS_XT30PW-M_1x02_P2.50mm_Horizontal, Connector_AMASS:AMASS_XT30PW-M_1x02_P2.50mm_Horizontal, F.Cu at (116.0, 101.0)
- added REF**: AMASS_XT30PW-M_1x02_P2.50mm_Horizontal, Connector_AMASS:AMASS_XT30PW-M_1x02_P2.50mm_Horizontal, F.Cu at (116.0, 86.5)
- added U203: TPS5460 康威科技, lib:TPS5460 康威科技, F.Cu at (72.9, 117.0)
- added U203: TPS5460 康威科技, lib:TPS5460 康威科技, F.Cu at (73.0, 72.8)
- R101, R102, R103: value 2k -> 10k
- moved C201 88.5 mm to (165.5, 66.4)
- moved C202 88.5 mm to (182.5, 66.4)
- moved C203 88.5 mm to (199.5, 66.4)
- moved C204 88.5 mm to (165.5, 81.4)
- moved C205 88.5 mm to (182.5, 81.4)
- moved C206 88.5 mm to (199.5, 81.4)
- moved C207 88.5 mm to (165.5, 96.4)
- moved C208 88.5 mm to (182.5, 96.4)
- moved C209 88.5 mm to (199.5, 96.4)
- moved G*** 86.5 mm to (167.6, 172.0) (x2)
- moved J201 83.5 mm to (-15.0, 60.5)
- moved J204 83.5 mm to (-15.0, 75.5)
- moved J205 83.5 mm to (2.00, 75.5)
- moved J206 83.5 mm to (19.0, 75.5)
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Connections:
- D104 pad 2: /relay_sig -> VCCF
Routing:
- net VCC: track 81.6 -> 0.00 mm
- net /relay_sig: track 72.2 -> 0.00 mm
- net V_{Comp}: track 34.5 -> 0.00 mm
- net Net-(D104-K): track 32.7 -> 0.00 mm
- net Net-(D103-K): track 20.7 -> 0.00 mm
- net Net-(D102-K): track 7.50 -> 0.00 mm
- net Net-(J106-Pin_3): track 2.54 -> 0.00 mm
- net Net-(J106-Pin_2): track 2.54 -> 0.00 mm
- net GND: vias 3 -> 0
- removed copper zone on F.Cu, net /VCC_FUSE
- removed copper zone on F.Cu, net VCC
- removed copper zone on F.Cu, net VCCF
Other:
- board size 80 x 80 mm -> 80 x 100 mm

Commit message: updated rev2
Parts:
- removed C101, C102, C103, C104, C105, C201, C202, C204: 560u, lib:CP_Radial_D10.0mm_P5.00mm
- removed the J201 at (-15.0, 60.5)
- removed the J204 at (-15.0, 75.5)
- removed REF** (x6): AMASS_XT30PW-M_1x02_P2.50mm_Horizontal, Connector_AMASS:AMASS_XT30PW-M_1x02_P2.50mm_Horizontal
- removed REF**: FUSE-MCCQ-121, lib:FUSE-MCCQ-121
- added F101: Fuse, lib:FUSE-MCCQ-121, F.Cu at (96.8, 134.8)
- added J214: VCC_{OUT}1, Connector_PinHeader_2.54mm:PinHeader_2x04_P2.54mm_Vertical, F.Cu at (52.9, 98.3)
- added J215: VCC_{OUT}2, Connector_PinHeader_2.54mm:PinHeader_2x04_P2.54mm_Vertical, F.Cu at (52.9, 105.5)
- added J216: VCCF, lib:AMASS_XT30U-F_1x02_P5.0mm_Vertical, F.Cu at (91.5, 98.0)
- D103: renamed from D104; value Green -> Red
- D104: renamed from D103; value Red -> Green
- J104: value Voltmeter Probe -> Voltmeter
- J201, J203: renamed from J202; value Power Out -> VCCF; footprint lib:AMASS_XT30U-M_1x02_P5.0mm_Vertical -> lib:AMASS_XT30PW-F_1x02_P2.50mm_Horizontal
- J202, J205, J206: value Power Out -> VCCF; footprint lib:AMASS_XT30U-M_1x02_P5.0mm_Vertical -> lib:AMASS_XT30PW-F_1x02_P2.50mm_Horizontal
- J204: renamed from J203; value Power Out -> VCCF; footprint lib:AMASS_XT30U-M_1x02_P5.0mm_Vertical -> lib:AMASS_XT30PW-F_1x02_P2.50mm_Horizontal
- J207, J208, J209: value Power Out -> VCCF; footprint lib:AMASS_XT30U-M_1x02_P5.0mm_Vertical -> lib:AMASS_XT30U-F_1x02_P5.0mm_Vertical
- J210: value 12v Out -> VCC_{OUT}1; footprint lib:AMASS_XT30U-M_1x02_P5.0mm_Vertical -> lib:AMASS_XT30PW-F_1x02_P2.50mm_Horizontal
- J211: value 12v Out -> VCC_{OUT}2; footprint lib:AMASS_XT30U-M_1x02_P5.0mm_Vertical -> lib:AMASS_XT30PW-F_1x02_P2.50mm_Horizontal
- J212: value 12v Out -> VCC_{OUT}1; footprint Connector_PinHeader_2.54mm:PinHeader_2x04_P2.54mm_Vertical -> lib:AMASS_XT30PW-F_1x02_P2.50mm_Horizontal
- J213: value 5v Out -> VCC_{OUT}2; footprint Connector_PinHeader_2.54mm:PinHeader_2x04_P2.54mm_Vertical -> lib:AMASS_XT30PW-F_1x02_P2.50mm_Horizontal
- moved J104 159.1 mm to (106.0, 144.5)
- moved G*** 146.1 mm to (66.0, 67.0), turned to 90 degrees
- moved G*** 146.1 mm to (66.0, 67.0), turned to -90 degrees
- moved C203 140.8 mm to (65.6, 110.0), turned to 0 degrees
- moved C206 139.5 mm to (65.8, 121.0), turned to 0 degrees
- moved C209 138.5 mm to (65.6, 132.0), turned to 0 degrees
- moved J213 134.1 mm to (60.1, 132.8), turned to 90 degrees
- moved J207 123.0 mm to (106.9, 107.0), turned to 0 degrees
- moved C205 113.0 mm to (76.6, 121.0), turned to 0 degrees
- moved C208 111.7 mm to (76.6, 132.0), turned to 0 degrees
- moved J211 110.6 mm to (60.1, 117.4), turned to 90 degrees
- moved J212 106.4 mm to (60.1, 88.6), turned to 90 degrees
- moved J205 97.6 mm to (98.5, 60.8), turned to 0 degrees
- moved R103 96.7 mm to (62.5, 140.2), turned to 0 degrees
- moved J102 95.7 mm to (74.8, 144.5)
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- renumbered U203 to U201, U203 to U202
Connections:
- D102 pad 2: VCC -> /VCC_FUSE
- D103 pad 1: Net-(D104-K) -> Net-(D103-K)
- D103 pad 2: VCCF -> V_{Comp}
- D104 pad 1: Net-(D103-K) -> Net-(D104-K)
- D104 pad 2: V_{Comp} -> VCCF
- J210 pad 2: +12V -> VCC_{OUT}1
- J211 pad 2: +12V -> VCC_{OUT}2
- J212 pad 2: +12V -> VCC_{OUT}1
- J213 pad 2: +5V -> VCC_{OUT}2
- U201 pad 1: (no net) -> VCCF
- U201 pad 2: (no net) -> VCC_{OUT}1
- U201 pad EN: (no net) -> unconnected-(U201-PadEN)
- U201 pad G: (no net) -> GND
- U202 pad 1: (no net) -> VCCF
- U202 pad 2: (no net) -> VCC_{OUT}2
- U202 pad EN: (no net) -> unconnected-(U202-PadEN)_1
- U202 pad G: (no net) -> GND
Routing:
- net /relay_sig: track 0.00 -> 39.2 mm
- net V_{Comp}: track 0.00 -> 27.4 mm
- net /VCC_FUSE: track 0.00 -> 26.4 mm
- net VCC: track 0.00 -> 15.3 mm
- net Net-(D103-K): track 0.00 -> 8.33 mm
- net Net-(D102-K): track 0.00 -> 8.31 mm
- net Net-(D104-K): track 0.00 -> 8.01 mm
- net Net-(J103-Pin_2): track 0.00 -> 2.54 mm
- net Net-(J103-Pin_3): track 0.00 -> 2.54 mm
- net GND: vias 0 -> 1
- added copper zone on F.Cu, net /VCC_FUSE
- added copper zone on F.Cu, net VCC
- added copper zone on F.Cu, net VCCF
- added copper zone on F.Cu, net VCC_{OUT}1
- added copper zone on F.Cu, net VCC_{OUT}2
Other:
- board text added: "POWER DISTRIBUTION UNIT HV R2"
- board text removed: "12V"
- board text removed: "14V60A"
- board text removed: "POWER DISTRIBUTION UNIT HV R1"
- board text removed: "Relay"
- board text removed: "Scott CJX"
- board text removed: "VCC"
- board text removed: "VComp"
