File: HDK/MecatronPDU-HV.kicad_sch (KiCad schematic)
At the start: 21 parts, among them J101 Power In, J102 V_{Comp}, J106 E-Stops, K101 Relay_SPST-NO

Commit message: init v2
Parts:
- added J104: Voltmeter Probe, lib:JST_XH_B2B-XH-AM_1x02_P2.50mm_Vertical, symbol Connector_Generic:Conn_01x02
- R101, R102, R103: value 2k -> 10k
- renumbered J106 to J103
Connections:
- net GND: now also J104.2 (Pin_2)
- net VCC: now also J104.1 (Pin_1)
- net VCCF: now also D104.2 (A)
- net relay_sig: no longer D104.2 (A)
Other:
- moved on the sheet: D103, D104, R102, R103

Commit message: updated rev2
Parts:
- removed C101, C102, C103, C104, C105: 560u, lib:CP_Radial_D10.0mm_P5.00mm, symbol Device:C_Polarized
- F101: footprint lib:FUSE-MCCQ-122 -> lib:FUSE-MCCQ-121
- J104: value Voltmeter Probe -> Voltmeter
Connections:
- net VCC: no longer D102.2 (A)
- net VCC_FUSE: now also D102.2 (A)
