File: HDK/Outputs.kicad_sch (KiCad schematic)
At the start: 18 parts, among them J201 Power Out, J202 Power Out, J203 Power Out, J204 Power Out, J205 Power Out, J206 Power Out, J207 Power Out, J208 Power Out, J209 Power Out

Commit message: init v2
Parts:
- removed J203: Power Out, lib:AMASS_XT30U-M_1x02_P5.0mm_Vertical, symbol Connector_Generic:Conn_01x02
- added J201: Power Out, lib:AMASS_XT30U-M_1x02_P5.0mm_Vertical, symbol Connector_Generic:Conn_01x02
- added J210, J211: 12v Out, lib:AMASS_XT30U-M_1x02_P5.0mm_Vertical, symbol Connector_Generic:Conn_01x02
- added J212: 12v Out, Connector_PinHeader_2.54mm:PinHeader_2x04_P2.54mm_Vertical, symbol Connector_Generic:Conn_02x04_Odd_Even
- added J213: 5v Out, Connector_PinHeader_2.54mm:PinHeader_2x04_P2.54mm_Vertical, symbol Connector_Generic:Conn_02x04_Odd_Even
- added U201, U202: TPS5460 康威科技, lib:TPS5460 康威科技, symbol scottcjx-kicad-lib:TPS5460 康威科技
- renumbered J201 to J202, J202 to J203
Connections:
- net GND: now also J201.1 (Pin_1), J210.1 (Pin_1), J211.1 (Pin_1), J212.1 (Pin_1), J212.3 (Pin_3), J212.5 (Pin_5), J212.7 (Pin_7), J213.1 (Pin_1), J213.3 (Pin_3), J213.5 (Pin_5), J213.7 (Pin_7), U201.G (GND), U202.G (GND)
- net VCCF: now also J201.2 (Pin_2), U201.1 (V_{IN}), U202.1 (V_{IN})
- new net +12V: J210.2 (Pin_2), J211.2 (Pin_2), J212.2 (Pin_2), J212.4 (Pin_4), J212.6 (Pin_6), J212.8 (Pin_8), U201.2 (V_{OUT})
- new net +5V: J213.2 (Pin_2), J213.4 (Pin_4), J213.6 (Pin_6), J213.8 (Pin_8), U202.2 (V_{OUT})
- no-connect marks 0 -> 2
Other:
- moved on the sheet: J202, J203

Commit message: updated rev2
Parts:
- added J211, J213: VCC_{OUT}2, lib:AMASS_XT30PW-F_1x02_P2.50mm_Horizontal, symbol Connector_Generic:Conn_01x02
- added J216: VCCF, lib:AMASS_XT30U-F_1x02_P5.0mm_Vertical, symbol Connector_Generic:Conn_01x02
- J201, J202, J203, J204, J205, J206: value Power Out -> VCCF; footprint lib:AMASS_XT30U-M_1x02_P5.0mm_Vertical -> lib:AMASS_XT30PW-F_1x02_P2.50mm_Horizontal
- J207, J208, J209: value Power Out -> VCCF; footprint lib:AMASS_XT30U-M_1x02_P5.0mm_Vertical -> lib:AMASS_XT30U-F_1x02_P5.0mm_Vertical
- J210: value 12v Out -> VCC_{OUT}1; footprint lib:AMASS_XT30U-M_1x02_P5.0mm_Vertical -> lib:AMASS_XT30PW-F_1x02_P2.50mm_Horizontal
- J212: renamed from J211; value 12v Out -> VCC_{OUT}1; footprint lib:AMASS_XT30U-M_1x02_P5.0mm_Vertical -> lib:AMASS_XT30PW-F_1x02_P2.50mm_Horizontal
- J214: renamed from J212; value 12v Out -> VCC_{OUT}1
- J215: renamed from J213; value 5v Out -> VCC_{OUT}2
Connections:
- net GND: now also J211.1 (Pin_1), J213.1 (Pin_1), J216.1 (Pin_1)
- net VCCF: now also J216.2 (Pin_2)
- net +12V renamed VCC_{OUT}1
- net +5V renamed VCC_{OUT}2
- net VCC_{OUT}2: now also J211.2 (Pin_2), J213.2 (Pin_2)
