File: HDK/esc-breakout/esc-breakout.kicad_pcb (KiCad board)
At the start: 2 copper layers, 80 x 30 mm, 13 parts, among them J101 Conn_PWR-OUT, J102 Conn_PWR-OUT, J103 Conn_PWR-OUT, J104 Conn_PWR-OUT, J105 Conn_PWR-OUT, J106 Conn_PWR-OUT, J107 Conn_PWR-OUT, J108 Conn_PWR-OUT, P101 Conn_PWR-IN

Commit message: rev3
Parts:
- added G***: LOGO, mecatron-logo-fp:mecatron-logo-fp30, F.Cu at (91.0, 65.0)
- added G***: LOGO, mecatron-logo-fp:mecatron-logo-fp30, B.Cu at (95.0, 65.0)
Other:
- board text added: "ESC BREAKOUT"
- board text added: "Scott CJX"
