File: HDK/pdu-hv-v3/HV-PDU-V3.kicad_pcb (KiCad board)
At the start: 2 copper layers, 80 x 100 mm, 29 parts, among them J101 Conn_PWR, J102 Conn_PWR, J103 Conn_01x03, J104 E-Stops, J105 Conn_PWR, K101 Relay_SPST-NO, U101 TPS5460 康威科技, U102 TPS5460 康威科技

Commit message: rev3
Parts:
- removed REF** (x2): AMASS_XT30UPB-F_1x02_P5.0mm_Vertical, scottcjx-kicad-lib:AMASS_XT30UPB-F_1x02_P5.0mm_Vertical
- removed REF** (x2): PinHeader_2x08_P2.54mm_Horizontal, Connector_PinHeader_2.54mm:PinHeader_2x08_P2.54mm_Horizontal
- added C110: 560u, scottcjx-kicad-lib:CP_Radial_D10.0mm_P5.00mm, F.Cu at (112.0, 65.5)
- added F101: Fuse, scottcjx-kicad-lib:FUSE-MCCQ-121, F.Cu at (115.0, 130.5)
- added G***: LOGO, mecatron-logo-fp:mecatron-logo-fp30, F.Cu at (94.0, 148.5)
- added J106: Conn_02x06_Odd_Even, Connector_PinHeader_2.54mm:PinHeader_2x06_P2.54mm_Vertical, F.Cu at (85.7, 143.0)
- added J107: Conn_02x06_Odd_Even, Connector_PinHeader_2.54mm:PinHeader_2x06_P2.54mm_Vertical, F.Cu at (67.2, 143.0)
- added J108: Conn_PWR, scottcjx-kicad-lib:AMASS_XT30UPB-F_1x02_P5.0mm_Vertical, F.Cu at (59.0, 123.0)
- added J109: Conn_PWR, scottcjx-kicad-lib:AMASS_XT30UPB-F_1x02_P5.0mm_Vertical, F.Cu at (59.0, 138.0)
- added J110: Conn_PWR, scottcjx-kicad-lib:AMASS_XT60-M_1x02_P7.20mm_Vertical, F.Cu at (99.0, 87.0)
- added J111: DMM, scottcjx-kicad-lib:JST_XH_B2B-XH-AM_1x02_P2.50mm_Vertical, F.Cu at (131.0, 143.0)
- added R101: 10k, Resistor_THT:R_Axial_DIN0207_L6.3mm_D2.5mm_P7.62mm_Horizontal, F.Cu at (124.0, 70.2)
- added R102: 10k, Resistor_THT:R_Axial_DIN0207_L6.3mm_D2.5mm_P7.62mm_Horizontal, F.Cu at (124.0, 89.8)
- added R103: 10k, Resistor_THT:R_Axial_DIN0207_L6.3mm_D2.5mm_P7.62mm_Horizontal, F.Cu at (124.0, 100.8)
- J101: moved to F.Cu
- J102: value Conn_PWR -> V_{COMP}
- moved D104 75.3 mm to (130.5, 75.3), turned to 90 degrees
- moved D103 65.0 mm to (130.5, 87.3), turned to 90 degrees
- moved C109 58.0 mm to (67.0, 87.5)
- moved C108 58.0 mm to (67.0, 76.5)
- moved C107 58.0 mm to (67.0, 65.4)
- moved D102 57.2 mm to (130.5, 98.3), turned to 90 degrees
- moved J104 54.3 mm to (131.5, 111.5), turned to 180 degrees
- moved J103 46.3 mm to (129.0, 115.5), turned to 0 degrees
- moved J102 45.2 mm to (131.0, 130.0), turned to -90 degrees
- moved U101 40.6 mm to (94.5, 115.8), turned to -90 degrees
- moved J105 34.5 mm to (98.6, 77.0), turned to 0 degrees
- moved C103 22.9 mm to (78.5, 87.5)
- moved C102 22.9 mm to (78.5, 76.5)
- moved C101 22.9 mm to (78.5, 65.4)
- moved D101 14.9 mm to (124.2, 115.2), turned to -90 degrees
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Connections:
- J103 pad 1: VCC -> VCCF
- U101 pad 1: VCCF -> VCCFR
- U102 pad 1: VCCF -> VCCFR
Routing:
- net VCCF: track 0.00 -> 78.1 mm
- net V_{Relay}: track 0.00 -> 32.9 mm
- net V_{Relay_Cont}: track 0.00 -> 19.5 mm
- net VCCFR: track 0.00 -> 16.9 mm, vias 0 -> 1
- net Net-(D104-A): track 0.00 -> 10.2 mm
- net V_{Comp}: track 0.00 -> 9.00 mm
- net Net-(D103-A): track 0.00 -> 7.55 mm
- net Net-(D102-A): track 0.00 -> 7.55 mm
- net Net-(J104-Pin_2): track 0.00 -> 2.54 mm
- net Net-(J104-Pin_3): track 0.00 -> 2.54 mm
- net GND: vias 0 -> 1
- added copper zone on B.Cu, net GND
- added copper zone on F.Cu, net GND
- added copper zone on B.Cu, net VCC
- added copper zone on F.Cu, net VCC
- added copper zone on B.Cu, net VCCF
- added copper zone on F.Cu, net VCCF
- added copper zone on F.Cu, net VCCFR
- added copper zone on F.Cu, net VCC_{OUT}1
- added copper zone on F.Cu, net VCC_{OUT}2
Other:
- board text added: "+"
- board text added: "DANGER ! HIGH VOLTAGE ! DANGER"
- board text added: "L"
- board text added: "POWER DISTRIBUTION UNIT HV R3"
- board text added: "R"
- board text added: "Scott CJX"
- board text added: "V_{CCFR}"
- board text added: "V_{CCF}"
- board text added: "V_{RELAY}SEL"
- board text added: "V_{Relay}"
