File: HDK/pdu-hv-v3/HV-PDU-V3.kicad_sch (KiCad schematic)
At the start: 29 parts, among them J101 Conn_PWR, J102 Conn_PWR, J103 Conn_01x03, J104 E-Stops, J105 Conn_PWR, K101 Relay_SPST-NO, U101 TPS5460 康威科技, U102 TPS5460 康威科技

Commit message: rev3
Parts:
- added C110: 560u, scottcjx-kicad-lib:CP_Radial_D10.0mm_P5.00mm, symbol Device:C_Polarized
- added J106, J107: Conn_02x06_Odd_Even, Connector_PinHeader_2.54mm:PinHeader_2x06_P2.54mm_Vertical, symbol Connector_Generic:Conn_02x06_Odd_Even
- added J108, J109: Conn_PWR, scottcjx-kicad-lib:AMASS_XT30UPB-F_1x02_P5.0mm_Vertical, symbol scottcjx-common-parts:Conn_+/-
- added J110: Conn_PWR, scottcjx-kicad-lib:AMASS_XT60-M_1x02_P7.20mm_Vertical, symbol scottcjx-common-parts:Conn_+/-
- added J111: DMM, scottcjx-kicad-lib:JST_XH_B2B-XH-AM_1x02_P2.50mm_Vertical, symbol scottcjx-common-parts:Conn_+/-
- F101: footprint (none) -> scottcjx-kicad-lib:FUSE-MCCQ-121
- J102: value Conn_PWR -> V_{COMP}
- R101, R102, R103: footprint (none) -> Resistor_THT:R_Axial_DIN0207_L6.3mm_D2.5mm_P7.62mm_Horizontal
Connections:
- net GND: now also C110.2, J106.1 (Pin_1), J106.11 (Pin_11), J106.3 (Pin_3), J106.5 (Pin_5), J106.7 (Pin_7), J106.9 (Pin_9), J107.1 (Pin_1), J107.11 (Pin_11), J107.3 (Pin_3), J107.5 (Pin_5), J107.7 (Pin_7), J107.9 (Pin_9), J108.- (Pin_2), J109.- (Pin_2), J110.- (Pin_2), J111.- (Pin_2)
- net VCC: no longer J103.1 (Pin_1)
- net VCCF: now also J103.1 (Pin_1), J111.+ (Pin_1); no longer U101.1 (V_{IN}), U102.1 (V_{IN})
- net VCCFR: now also U101.1 (V_{IN}), U102.1 (V_{IN}), C110.1, J110.+ (Pin_1)
- net VCC_{OUT}1: now also J106.10 (Pin_10), J106.12 (Pin_12), J106.2 (Pin_2), J106.4 (Pin_4), J106.6 (Pin_6), J106.8 (Pin_8), J108.+ (Pin_1)
- net VCC_{OUT}2: now also J107.10 (Pin_10), J107.12 (Pin_12), J107.2 (Pin_2), J107.4 (Pin_4), J107.6 (Pin_6), J107.8 (Pin_8), J109.+ (Pin_1)
